File: pcb/pcb.kicad_sch (KiCad schematic)
At the start: 0 parts

Commit message: making the schematic
Parts:
- added D1, D2, D3, D4, D5, D6, D7, D8, D9: 1N4148, Diode_THT:D_DO-35_SOD27_P7.62mm_Horizontal, symbol Diode:1N4148
- added SW1, SW2, SW3, SW4, SW5, SW6, SW7, SW8, SW9: SW_Push, Button_Switch_Keyboard:SW_Cherry_MX_1.00u_PCB, symbol Switch:SW_Push
- added SW10: RotaryEncoder_Switch, Rotary_Encoder:RotaryEncoder_Alps_EC11E-Switch_Vertical_H20mm, symbol Device:RotaryEncoder_Switch
- added U1: MOUDLE-SEEEDUINO-XIAO, footprints:XIAO-Generic-Hybrid-14P-2.54-21X17.8MM, symbol XIAO_RP2040:MOUDLE-SEEEDUINO-XIAO
- added U2: ER_OLEDM0.91_1x-I2C, Display:ER_OLEDM0.91_1x-I2C, symbol Display_Graphic:ER_OLEDM0.91_1x-I2C
Connections:
- new net: D1.2 (A), SW1.2
- new net: D4.2 (A), SW4.2
- new net: D5.2 (A), SW5.2
- new net: D3.2 (A), SW3.2
- new net: D7.2 (A), SW7.2
- new net: D8.2 (A), SW8.2
- new net: D2.2 (A), SW2.2
- new net: D6.2 (A), SW6.2
- new net: D9.2 (A), SW9.2
- new net C1: SW1.1, SW4.1, SW7.1, U1.7 (PB08_A6_D6_TX)
- new net C2: SW2.1, SW5.1, SW8.1, U1.8 (PB09_A7_D7_RX)
- new net C3: SW3.1, SW6.1, SW9.1, U1.9 (PA7_A8_D8_SCK)
- new net GND: SW10.C, SW10.S2, U1.13 (GND), U2.1 (GND)
- new net R1: D1.1 (K), D2.1 (K), D3.1 (K), U1.1 (PA02_A0_D0)
- new net R2: D4.1 (K), D5.1 (K), D6.1 (K), U1.2 (PA4_A1_D1)
- new net R3: D7.1 (K), D8.1 (K), D9.1 (K), U1.3 (PA10_A2_D2)
- new net RE1: SW10.A, U1.10 (PA5_A9_D9_MISO)
- new net RE2: SW10.B, U1.11 (PA6_A10_D10_MOSI)
- new net RE3: SW10.S1, U1.4 (PA11_A3_D3)
- new net SCL: U1.6 (PA9_A5_D5_SCL), U2.3 (SCL)
- new net SDA: U1.5 (PA8_A4_D4_SDA), U2.4 (SDA)
- new net VCC: U1.14 (5V), U2.2 (VCC)
Other:
- company: (none) -> Jishnu Dutta
- title: (none) -> ByteBoard

Commit message: making the schematic and adding assets
Parts:
- SW1, SW2, SW3, SW4, SW5, SW6, SW7, SW8, SW9: footprint Button_Switch_Keyboard:SW_Cherry_MX_1.00u_PCB -> JishnuKey:SW_Cherry_MX_1.00u_PCB_Custom
Changed lines of the file:
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@@
 			)
 		)
-		(property "Footprint" "Button_Switch_Keyboard:SW_Cherry_MX_1.00u_PCB"
+		(property "Footprint" "JishnuKey:SW_Cherry_MX_1.00u_PCB_Custom"
 			(at 177.8 119.38 0)
 			(hide yes)
@@
 			)
 		)
-		(property "Footprint" "Button_Switch_Keyboard:SW_Cherry_MX_1.00u_PCB"
+		(property "Footprint" "JishnuKey:SW_Cherry_MX_1.00u_PCB_Custom"
 			(at 156.21 99.06 0)
 			(hide yes)
@@
 			)
 		)
-		(property "Footprint" "Button_Switch_Keyboard:SW_Cherry_MX_1.00u_PCB"
+		(property "Footprint" "JishnuKey:SW_Cherry_MX_1.00u_PCB_Custom"
 			(at 199.39 99.06 0)
 			(hide yes)
@@
 			)
 		)
-		(property "Footprint" "Button_Switch_Keyboard:SW_Cherry_MX_1.00u_PCB"
+		(property "Footprint" "JishnuKey:SW_Cherry_MX_1.00u_PCB_Custom"
 			(at 156.21 137.16 0)
 			(hide yes)
@@
 			)
 		)
-		(property "Footprint" "Button_Switch_Keyboard:SW_Cherry_MX_1.00u_PCB"
+		(property "Footprint" "JishnuKey:SW_Cherry_MX_1.00u_PCB_Custom"
 			(at 156.21 119.38 0)
 			(hide yes)
@@
 			)
 		)
-		(property "Footprint" "Button_Switch_Keyboard:SW_Cherry_MX_1.00u_PCB"
+		(property "Footprint" "JishnuKey:SW_Cherry_MX_1.00u_PCB_Custom"
 			(at 177.8 137.16 0)
 			(hide yes)
@@
 			)
 		)
-		(property "Footprint" "Button_Switch_Keyboard:SW_Cherry_MX_1.00u_PCB"
+		(property "Footprint" "JishnuKey:SW_Cherry_MX_1.00u_PCB_Custom"
 			(at 199.39 119.38 0)
 			(hide yes)
@@
 			)
 		)
-		(property "Footprint" "Button_Switch_Keyboard:SW_Cherry_MX_1.00u_PCB"
+		(property "Footprint" "JishnuKey:SW_Cherry_MX_1.00u_PCB_Custom"
 			(at 199.39 137.16 0)
 			(hide yes)
@@
 			)
 		)
-		(property "Footprint" "Button_Switch_Keyboard:SW_Cherry_MX_1.00u_PCB"
+		(property "Footprint" "JishnuKey:SW_Cherry_MX_1.00u_PCB_Custom"
 			(at 177.8 99.06 0)
 			(hide yes)

Commit message: routing on the pcb
Parts:
- added D10, D11, D12, D13, D14, D15, D16, D17, D18: SK6812MINI-E, LED_SMD:LED_SK6812MINI-E_3.2x2.8mm_P1.5mm_ReverseMount, symbol LED:SK6812MINI-E
- added H1, H2, H3, H4: MountingHole, MountingHole:MountingHole_3.2mm_M3, symbol Mechanical:MountingHole
- D1, D2, D3, D4, D5, D6, D7, D8, D9: KiLib_Generator (none) -> diode/THT
Connections:
- net GND: now also D10.1 (VSS), D11.1 (VSS), D12.1 (VSS), D13.1 (VSS), D14.1 (VSS), D15.1 (VSS), D16.1 (VSS), D17.1 (VSS), D18.1 (VSS); no longer SW10.S2
- net VCC: now also D10.3 (VDD), D11.3 (VDD), D12.3 (VDD), D13.3 (VDD), D14.3 (VDD), D15.3 (VDD), D16.3 (VDD), D17.3 (VDD), D18.3 (VDD)
- net RE3: no longer names the net of SW10.S1
- net RE3: no longer U1.4 (PA11_A3_D3)
- new net: D12.4 (DOUT), D13.2 (DIN)
- new net: D13.4 (DOUT), D14.2 (DIN)
- new net: D10.4 (DOUT), D11.2 (DIN)
- new net: D11.4 (DOUT), D12.2 (DIN)
- new net: D14.4 (DOUT), D15.2 (DIN)
- new net: D15.4 (DOUT), D16.2 (DIN)
- new net: D16.4 (DOUT), D17.2 (DIN)
- new net: D17.4 (DOUT), D18.2 (DIN)
- new net RGB: D10.2 (DIN), U1.4 (PA11_A3_D3)
