File: pcb/pcb.kicad_pcb (KiCad board)
At the start: 2 copper layers, 21 parts, among them SW1 SW_Push, SW10 RotaryEncoder_Switch, SW2 SW_Push, SW3 SW_Push, SW4 SW_Push, SW5 SW_Push, SW6 SW_Push, SW7 SW_Push, SW8 SW_Push, SW9 SW_Push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

Commit message: making the schematic and adding assets
Parts:
- SW1, SW2, SW3, SW4, SW5, SW6, SW7, SW8, SW9: footprint Button_Switch_Keyboard:SW_Cherry_MX_1.00u_PCB -> JishnuKey:SW_Cherry_MX_1.00u_PCB_Custom
- moved U1 106.5 mm to (90.4, 38.6)
- moved D7 87.5 mm to (87.5, 125.5)
- moved D4 82.4 mm to (86.7, 98.0)
- moved SW10 80.2 mm to (106.5, 37.6)
- moved D1 78.8 mm to (87.9, 72.5)
- moved SW7 75.3 mm to (89.5, 116.5), turned to 180 degrees
- moved D8 59.3 mm to (117.7, 125.0)
- moved D5 51.6 mm to (117.7, 97.5)
- moved D2 50.0 mm to (116.5, 72.5)
- moved SW4 48.4 mm to (88.9, 90.6), turned to 180 degrees
- moved SW8 44.4 mm to (118.4, 116.6), turned to 180 degrees
- moved SW3 43.5 mm to (145.5, 65.1), turned to 180 degrees
- moved D9 36.8 mm to (145.5, 125.0)
- moved U2 35.5 mm to (127.0, 44.0), turned to 90 degrees
- moved SW1 26.6 mm to (89.5, 65.1), turned to 180 degrees
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
Commit message: routing on the pcb
Parts:
- added D10: SK6812MINI-E, LED_SMD:LED_SK6812MINI-E_3.2x2.8mm_P1.5mm_ReverseMount, B.Cu at (92.2, 52.8)
- added D11: SK6812MINI-E, LED_SMD:LED_SK6812MINI-E_3.2x2.8mm_P1.5mm_ReverseMount, B.Cu at (111.3, 52.8)
- added D12: SK6812MINI-E, LED_SMD:LED_SK6812MINI-E_3.2x2.8mm_P1.5mm_ReverseMount, B.Cu at (130.0, 52.8)
- added D13: SK6812MINI-E, LED_SMD:LED_SK6812MINI-E_3.2x2.8mm_P1.5mm_ReverseMount, B.Cu at (92.2, 72.2)
- added D14: SK6812MINI-E, LED_SMD:LED_SK6812MINI-E_3.2x2.8mm_P1.5mm_ReverseMount, B.Cu at (111.3, 72.2)
- added D15: SK6812MINI-E, LED_SMD:LED_SK6812MINI-E_3.2x2.8mm_P1.5mm_ReverseMount, B.Cu at (130.2, 72.2)
- added D16: SK6812MINI-E, LED_SMD:LED_SK6812MINI-E_3.2x2.8mm_P1.5mm_ReverseMount, B.Cu at (92.2, 91.8)
- added D17: SK6812MINI-E, LED_SMD:LED_SK6812MINI-E_3.2x2.8mm_P1.5mm_ReverseMount, B.Cu at (111.3, 91.8)
- added D18: SK6812MINI-E, LED_SMD:LED_SK6812MINI-E_3.2x2.8mm_P1.5mm_ReverseMount, B.Cu at (130.0, 90.8)
- added H1: MountingHole, MountingHole:MountingHole_3.2mm_M3, F.Cu at (76.0, 30.0)
- added H2: MountingHole, MountingHole:MountingHole_3.2mm_M3, F.Cu at (76.0, 108.0)
- added H3: MountingHole, MountingHole:MountingHole_3.2mm_M3, F.Cu at (160.0, 30.0)
- added H3: MountingHole, MountingHole:MountingHole_3.2mm_M3, F.Cu at (160.0, 107.0)
- moved D9 25.3 mm to (127.2, 107.5)
- moved SW9 23.2 mm to (127.5, 103.1)
- moved D6 20.9 mm to (126.2, 87.5)
- moved D8 20.8 mm to (106.4, 107.5)
- moved D3 20.5 mm to (125.5, 69.0)
- moved SW6 19.4 mm to (127.4, 84.1)
- moved D7 18.0 mm to (87.7, 107.5)
- moved SW3 18.0 mm to (127.5, 65.1)
- moved SW8 16.8 mm to (108.4, 103.1)
- moved D5 13.8 mm to (107.2, 88.5)
- moved SW7 13.4 mm to (89.5, 103.1)
- moved SW5 11.4 mm to (108.4, 84.1)
- moved D2 9.95 mm to (107.2, 69.0)
- moved D4 9.59 mm to (88.0, 88.5)
- moved SW2 9.50 mm to (108.5, 65.1)
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Connections:
- SW10 pad S1: /RE3 -> unconnected-(SW10-PadS1)
- SW10 pad S2: GND -> unconnected-(SW10-PadS2)
- U1 pad 4: /RE3 -> /RGB
Routing:
- net VCC: track 0.00 -> 264.7 mm, vias 0 -> 16
- net GND: track 0.00 -> 242.6 mm, vias 0 -> 4
- net /R3: track 0.00 -> 135.2 mm
- net /R2: track 0.00 -> 112.4 mm, vias 0 -> 2
- net /C2: track 0.00 -> 101.3 mm
- net /R1: track 0.00 -> 84.2 mm, vias 0 -> 3
- net /C3: track 0.00 -> 83.9 mm, vias 0 -> 1
- net Net-(D12-DOUT): track 0.00 -> 71.9 mm
- net /C1: track 0.00 -> 59.1 mm
- net Net-(D17-DOUT): track 0.00 -> 53.0 mm, vias 0 -> 2
- net Net-(D11-DOUT): track 0.00 -> 51.0 mm, vias 0 -> 4
- net /SCL: track 0.00 -> 50.8 mm
- net /SDA: track 0.00 -> 48.4 mm
- net Net-(D10-DOUT): track 0.00 -> 46.7 mm
- net Net-(D15-DOUT): track 0.00 -> 46.2 mm, vias 0 -> 4
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Other:
- board outline added: 94 x 87.5 mm

Commit message: add readme and logo
Other:
- board text added: "<ByteBoard /> v1.0 Designed By Jishnu Dutta • 2026"
- board text added: "HACK CLUB"

Commit message: update Journal
Other:
- board size 94 x 87.5 mm -> 94 x 84.5 mm
Changed lines of the file:
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@@
 		(filling no)
 		(pcbplotparams
-			(layerselection 0x00000000_00000000_55555555_5755f5ff)
+			(layerselection 0x00000000_00000000_55555555_575555ff)
 			(plot_on_all_layers_selection 0x00000000_00000000_00000000_00000000)
 			(disableapertmacros no)
@@
 			(outputformat 1)
 			(mirror no)
-			(drillshape 1)
+			(drillshape 0)
 			(scaleselection 1)
-			(outputdirectory "")
+			(outputdirectory "gerber")
 		)
 	)
@@
 	)
 	(gr_rect
-		(start 71 25.259779)
-		(end 165 112.740221)
+		(start 71 26.999999)
+		(end 165 111.499999)
 		(stroke
 			(width 0.05)
@@
 		(layer "Edge.Cuts")
 	)
-	(gr_text "<ByteBoard /> v1.0\nDesigned By Jishnu Dutta • 2026"
-		(at 117 30.5 0)
-		(layer "F.Cu")
+	(gr_text "<ByteBoard /> v1.0\nDesigned By Jishnu Dutta \n• 2026"
+		(at 140.5 68 0)
+		(layer "F.SilkS")
 		(effects
 			(font
-				(size 1.5 1.5)
-				(thickness 0.3)
+				(size 1.2 1.2)
+				(thickness 0.25)
 				(bold yes)
 			)
@@
 	(gr_text "HACK CLUB"
 		(at 147 84.5 0)
-		(layer "F.Cu")
+		(layer "F.SilkS")
 		(effects
 			(font
